File: robocup2025_kicad_data.kicad_pcb (KiCad board)
At the start: 4 copper layers, 88.1 x 96.9 mm, 19 parts, among them M7 Motor_Servo, U2 ESP32-DEVKITC-32E

Commit message: new schematics and pcbs
Parts:
- added R2: 220, Resistor_THT:R_Axial_DIN0204_L3.6mm_D1.6mm_P7.62mm_Horizontal, F.Cu at (180.4, 115.0)
- added R3: 2.2k, Resistor_THT:R_Axial_DIN0204_L3.6mm_D1.6mm_P7.62mm_Horizontal, F.Cu at (180.4, 120.5)
- added U1: ~, robo:AE-BNO055-BO, F.Cu at (170.9, 49.4)
- moved M1 29.8 mm to (156.5, 85.5)
- moved M2 27.9 mm to (156.5, 91.0)
- moved M3 25.6 mm to (156.5, 96.0)
- moved U6 25.0 mm to (109.5, 91.4), turned to 90 degrees
- moved M4 23.8 mm to (156.5, 101.5)
- moved S1 23.3 mm to (166.5, 126.5)
- moved M5 21.9 mm to (156.5, 107.0)
- moved M7 15.0 mm to (154.5, 112.5)
- moved U3 7.25 mm to (172.4, 88.5)
- moved U4 7.25 mm to (172.4, 93.9)
- moved U5 7.25 mm to (172.4, 99.2)
- moved U2 3.50 mm to (127.8, 82.3)
- moved R1 1.00 mm to (168.4, 118.5)
Connections:
- R1 pad 1: ESP32_21 -> ESP32_25
- S1 pad 1: ESP32_21 -> ESP32_25
- U2 pad J2_8: unconnected-(U2-IO33-PadJ2_8) -> ultrasonic_trig2
- U2 pad J2_9: unconnected-(U2-IO25-PadJ2_9) -> ESP32_25
- U2 pad J3_3: ultrasonic_trig2 -> ESP32_22/SCL
- U2 pad J3_6: ESP32_21 -> ESP32_21/SDA
Routing:
- net ESP32_3.3: track 124.3 -> 0.00 mm, vias 3 -> 0
- net arm_feedback: track 97.6 -> 0.00 mm
- net tyre_pulse_2: track 90.8 -> 0.00 mm
- net ultrasonic_trig3: track 90.1 -> 0.00 mm
- net tyre_pulse_1: track 81.7 -> 0.00 mm, vias 1 -> 0
- net ultrasonic_echo3: track 81.1 -> 0.00 mm, vias 2 -> 0
- net ultrasonic_echo2: track 69.0 -> 0.00 mm
- net ESP32_21: track 68.8 -> 0.00 mm
- net Net-(L1-+): track 67.6 -> 0.00 mm
- net arm_wire_SIG: track 59.2 -> 0.00 mm, vias 1 -> 0
- net ultrasonic_trig2: track 54.6 -> 0.00 mm, vias 1 -> 0
- net ultrasonic_echo1: track 51.4 -> 0.00 mm
- net arm_pulse: track 45.7 -> 0.00 mm, vias 2 -> 0
- net ultrasonic_trig1: track 45.3 -> 0.00 mm, vias 1 -> 0
- net ESP32_5V: track 41.8 -> 0.00 mm
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Other:
- board text added: "TECHNOTORQUES テクノトルクス"
- board text added: "Voltage Meter"

Commit message: adding routed pcb
Routing:
- net ESP32_3.3: track 0.00 -> 167.0 mm
- net ESP32_21/SDA: track 0.00 -> 122.0 mm, vias 0 -> 1
- net arm_feedback: track 0.00 -> 116.8 mm, vias 0 -> 1
- net ultrasonic_trig2: track 0.00 -> 114.4 mm, vias 0 -> 1
- net ESP32_22/SCL: track 0.00 -> 106.2 mm
- net ultrasonic_trig3: track 0.00 -> 100.6 mm, vias 0 -> 2
- net ESP32_25: track 0.00 -> 99.8 mm, vias 0 -> 1
- net tyre_pulse_2: track 0.00 -> 93.2 mm, vias 0 -> 4
- net Net-(L1-+): track 0.00 -> 91.9 mm, vias 0 -> 1
- net ultrasonic_echo3: track 0.00 -> 73.0 mm
- net tyre_pulse_1: track 0.00 -> 68.6 mm, vias 0 -> 2
- net arm_wire_SIG: track 0.00 -> 67.0 mm, vias 0 -> 1
- net ultrasonic_echo2: track 0.00 -> 56.2 mm, vias 0 -> 1
- net arm_pulse: track 0.00 -> 48.2 mm
- net ESP32_5V: track 0.00 -> 44.2 mm
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